File: pcb-batterypack.kicad_sch (KiCad schematic)
At the start: 11 parts, among them J1 BATT_CON, J2 246, J3 246

Commit message: refactor battery pack edge cuts outline
Connections:
- net BATP: now also J1.3 (Pin_3); no longer J1.1 (Pin_1)
- net GND: now also J1.1 (Pin_1); no longer J1.3 (Pin_3)
Other:
- note added: "NOTE: Since a straight cable is used this pin layout is mirrored compared to the one on the MrHat pcb"
Changed lines of the file:
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@@
+		)
+	)
+	(text "NOTE: Since a straight cable is used\nthis pin layout is mirrored compared to the one on the MrHat pcb"
+		(exclude_from_sim no)
+		(at 183.896 90.932 0)
+		(effects
+			(font
+				(size 1.27 1.27)
+			)
 		)
 	)
@@
 		(lib_id "Connector_Generic:Conn_01x03")
 		(at 181.61 101.6 0)
+		(mirror x)
 		(unit 1)
 		(exclude_from_sim no)
@@
 		(on_board yes)
 		(dnp no)
-		(fields_autoplaced yes)
 		(property "Reference" "J1"
-			(at 184.15 100.3299 0)
+			(at 184.15 102.8701 0)
 			(effects
 				(font
@@
 		)
 		(property "Value" "BATT_CON"
-			(at 184.15 102.8699 0)
+			(at 184.15 100.3301 0)
 			(effects
 				(font
